File: Cubesat-Production/Power PCB/V_Reg_3.3V.kicad_sch (KiCad schematic)
At the start: 5 parts, among them U5 MAX710ESE+T

Commit message: Added missing component values
Parts:
- C29: value C_Polarized_US -> 4.7u
- C30: value C_Polarized_US -> 100u
- L5: value L -> 22u
Changed lines of the file:
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@@
       (effects (font (size 1.27 1.27)) (justify left))
     )
-    (property "Value" "C_Polarized_US" (id 1) (at 153.035 64.77 0)
+    (property "Value" "100u" (id 1) (at 153.035 64.77 0)
       (effects (font (size 1.27 1.27)) (justify left))
     )
@@
       (effects (font (size 1.27 1.27)) (justify left))
     )
-    (property "Value" "C_Polarized_US" (id 1) (at 136.525 76.2 0)
+    (property "Value" "4.7u" (id 1) (at 136.525 76.2 0)
       (effects (font (size 1.27 1.27)) (justify left))
     )
@@
     (in_bom yes) (on_board yes)
     (property "Reference" "L5" (id 0) (at 99.06 44.45 90))
-    (property "Value" "L" (id 1) (at 99.06 41.275 90))
+    (property "Value" "22u" (id 1) (at 99.06 41.275 90))
     (property "Footprint" "Inductor_SMD:L_0603_1608Metric_Pad1.05x0.95mm_HandSolder" (id 2) (at 99.06 43.18 0)
       (effects (font (size 1.27 1.27)) hide)
