File: Cubesat-Previous/Power PCB/CubesatPwrBoard.kicad_sch (KiCad schematic)
At the start: 53 parts, among them J1 SystemLoad, J10 Test_Point, J11 Test_Point, J14 Test_Point, J15 Test_Point, J16 Test_Point_GND, J2 SystemLoad, J3 I2C, J6 Test_Point, J7 Test_Point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

Commit message: moving prod to prev revision branch
Parts:
- removed BT7, BT8: 254TR, 254TR:BAT_254TR, symbol 254TR:254TR
- removed C1: 150u, Capacitor_SMD:C_0603_1608Metric_Pad1.08x0.95mm_HandSolder, symbol CubesatPwrBoard-rescue:CP1-Device
- removed C2: 0.1u, Capacitor_SMD:C_0603_1608Metric_Pad1.08x0.95mm_HandSolder, symbol CubesatPwrBoard-rescue:CP1-Device
- removed C3: 1u, Capacitor_SMD:C_0603_1608Metric_Pad1.08x0.95mm_HandSolder, symbol CubesatPwrBoard-rescue:C-Device
- removed C4: 4.7u, Capacitor_SMD:C_0603_1608Metric_Pad1.08x0.95mm_HandSolder, symbol CubesatPwrBoard-rescue:C-Device
- removed C5: 22n, Capacitor_SMD:C_0603_1608Metric_Pad1.08x0.95mm_HandSolder, symbol CubesatPwrBoard-rescue:C-Device
- removed C6, C7: 10u, Capacitor_SMD:C_0603_1608Metric_Pad1.08x0.95mm_HandSolder, symbol CubesatPwrBoard-rescue:C-Device
- removed D1, D2, D3, D4, D5, D6: D_Schottky_Small, CUS520,H3F:DIO_CUS520,H3F, symbol CubesatPwrBoard-rescue:D_Schottky_Small-Device
- removed J1, J2: SystemLoad, Connector_Wire:SolderWirePad_1x01_SMD_5x10mm, symbol CubesatPwrBoard-rescue:Conn_01x01_Female-Connector
- removed J10, J11, J14, J15, J6, J7: Test_Point, TestPoint:TestPoint_Pad_2.0x2.0mm, symbol CubesatPwrBoard-rescue:Conn_01x01_Female-Connector
- removed J16: Test_Point_GND, TestPoint:TestPoint_Pad_2.0x2.0mm, symbol CubesatPwrBoard-rescue:Conn_01x01_Female-Connector
- removed L1: 4.7u, Inductor_SMD:L_0603_1608Metric_Pad1.05x0.95mm_HandSolder, symbol CubesatPwrBoard-rescue:L-Device
- removed Q1: TQM110NB04CR_RLG, TQM110N:TRANS_TQM110NB04CR_RLG, symbol TQM110NB04CR_RLG:TQM110NB04CR_RLG
- removed Q2: 2N7002*, 2N7002:SOT23, symbol 2N7002_:2N7002*
- removed R1: 2.5, Resistor_SMD:R_0603_1608Metric_Pad0.98x0.95mm_HandSolder, symbol CubesatPwrBoard-rescue:R-Device
- removed R2, R3: 16m, Resistor_SMD:R_0603_1608Metric_Pad0.98x0.95mm_HandSolder, symbol CubesatPwrBoard-rescue:R-Device
- removed R4: 63.4k, Resistor_SMD:R_0603_1608Metric_Pad0.98x0.95mm_HandSolder, symbol CubesatPwrBoard-rescue:R-Device
- removed R5: 10m, Resistor_SMD:R_0603_1608Metric_Pad0.98x0.95mm_HandSolder, symbol CubesatPwrBoard-rescue:R-Device
- removed SC1, SC10, SC11, SC12, SC2, SC3, SC4, SC5, SC6, SC7, SC8, SC9: Solar_Cells, 6915_1x2:691508110302, symbol CubesatPwrBoard-rescue:Solar_Cells-Device
- removed TH1: Thermistor_NTC, Jumper:SolderJumper-2_P1.3mm_Open_Pad1.0x1.5mm, symbol CubesatPwrBoard-rescue:Thermistor_NTC-Device
- removed U1: LTC4162, LTC4162:QFN50P500X400X80-29N, symbol LTC4162IUFD:LTC4162
- added H1, H2, H3, H4: MountingHole_Pad, MountingHole:MountingHole_4.3mm_M4_DIN965_Pad, symbol Mechanical:MountingHole_Pad
- added J2, J3: Conn_01x04_Female, Connector_PinSocket_2.54mm:PinSocket_1x04_P2.54mm_Vertical, symbol Connector:Conn_01x04_Female
- added J5: Conn_01x04_Female, Connector_PinSocket_2.54mm:PinSocket_1x03_P2.54mm_Vertical, symbol Connector:Conn_01x03_Female
- added J6, J7, J8: Conn_01x03_Female, Connector_PinSocket_2.54mm:PinSocket_1x03_P2.54mm_Vertical, symbol Connector:Conn_01x03_Female
- added TH1, TH2, TH3: Thermistor_NTC, Resistor_SMD:R_0402_1005Metric_Pad0.72x0.64mm_HandSolder, symbol Device:Thermistor_NTC
- J1: renamed from J3; value I2C -> Conn_01x04_Female; footprint 6915_1x4:691508110304 -> Connector_PinSocket_2.54mm:PinSocket_1x04_P2.54mm_Vertical; symbol CubesatPwrBoard-rescue:Conn_01x04_Female-Connector -> Connector:Conn_01x04_Female
Connections:
- net GND: now also H1.1, H2.1, H3.1, H4.1, TH1.2, TH2.2, TH3.2
- net Bat_Reg_1//SMBALERT: now reaches J1.4 (Pin_4)
- net Bat_Reg_1/SCL: now reaches J1.3 (Pin_3)
- net Bat_Reg_1/SDA: now reaches J1.2 (Pin_2)
- net Bat_Reg_1/DVCC: now reaches J1.1 (Pin_1)
- new net Bat_Reg_1/TH: TH1.1
- new net Bat_Reg_1/V_Bat: BT1.P1_1, BT1.P1_2
- new net Bat_Reg_2/DVCC: J3.1 (Pin_1)
- new net Bat_Reg_2/SCL: J3.3 (Pin_3)
- new net Bat_Reg_2/SDA: J3.2 (Pin_2)
- new net Bat_Reg_2/TH: TH2.1
- new net Bat_Reg_2/V_Bat: BT3.P1_1, BT3.P1_2
- new net Bat_Reg_2//SMBALERT: J3.4 (Pin_4)
- new net Bat_Reg_3/DVCC: J2.1 (Pin_1)
- new net Bat_Reg_3/SCL: J2.3 (Pin_3)
- new net Bat_Reg_3/SDA: J2.2 (Pin_2)
- new net Bat_Reg_3/TH: TH3.1
- new net Bat_Reg_3/V_Bat: BT5.P1_1, BT5.P1_2
- new net Bat_Reg_3//SMBALERT: J2.4 (Pin_4)
- new net V_Reg_3.3_5V1/#SHDN: J6.3 (Pin_3)
- new net V_Reg_3.3_5V1/#STBY: J6.2 (Pin_2)
- new net V_Reg_3.3_5V1/3/#5: J6.1 (Pin_1)
- new net V_Reg_3.3_5V1/Vout: J5.1 (Pin_1)
- new net V_Reg_3.3_5V2/#SHDN: J8.3 (Pin_3)
- new net V_Reg_3.3_5V2/#STBY: J8.2 (Pin_2)
- new net V_Reg_3.3_5V2/3/#5: J8.1 (Pin_1)
- new net V_Reg_3.3_5V2/Vout: J5.2 (Pin_2)
- new net V_Reg_3.3_5V3/#SHDN: J7.3 (Pin_3)
- new net V_Reg_3.3_5V3/#STBY: J7.2 (Pin_2)
- new net V_Reg_3.3_5V3/3/#5: J7.1 (Pin_1)
- new net V_Reg_3.3_5V3/Vout: J5.3 (Pin_3)
Other:
- added sheet Bat_Reg_1 (Bat_Reg_1.kicad_sch)
- added sheet Bat_Reg_2 (Bat_Reg_1.kicad_sch)
- added sheet Bat_Reg_3 (Bat_Reg_1.kicad_sch)
- added sheet Solar_Panels (Solar_Panels.kicad_sch)
- added sheet V_Reg_3.3_5V1 (V_Reg_3.3V.kicad_sch)
- added sheet V_Reg_3.3_5V2 (V_Reg_3.3V.kicad_sch)
- added sheet V_Reg_3.3_5V3 (V_Reg_3.3V.kicad_sch)
- note added: "Each battery gets its own PMIC regulating voltage and its own I2C port for management"
- note removed: "Two solar cell groups per side - 12 total cell groups"
- moved on the sheet: BT1, BT2, J1
