File: Cubesat-Current/Power PCB/Bat_Reg_1.kicad_sch (KiCad schematic)
At the start: 16 parts, among them Q1 TQM110NB04CR_RLG, Q2 2N7002*, U1 LTC4162

Commit message: Fixed footprint size of 150uF caps
Parts:
- C1: footprint Capacitor_SMD:C_0603_1608Metric_Pad1.08x0.95mm_HandSolder -> Capacitor_SMD:C_1210_3225Metric_Pad1.33x2.70mm_HandSolder
Changed lines of the file:
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@@
       (effects (font (size 1.27 1.27)) (justify left))
     )
-    (property "Footprint" "Capacitor_SMD:C_0603_1608Metric_Pad1.08x0.95mm_HandSolder" (id 2) (at 60.96 60.96 0)
+    (property "Footprint" "Capacitor_SMD:C_1210_3225Metric_Pad1.33x2.70mm_HandSolder" (id 2) (at 60.96 60.96 0)
       (effects (font (size 1.27 1.27)) hide)
     )

Commit message: Updating to revision 5.0
Parts:
- C1: value C_Polarized_US -> 150u
- C2: value C_Polarized_US -> 0.1u
- C3: value C -> 1u
- C4: value C -> 4.7u
- C5: value C -> 22n
- C6, C7: value C -> 10u
- L1: value L -> 4.7u
- Q2: footprint 2N7002:SOT23 -> Connectors_Cubesat_Custom:CubeSat_2n7002
- R1: value R -> 2.5
- R2: value R -> 10k
- R3: value R -> 16m
- R4: value R -> 63.4k
- R5: value R -> 10m
Connections:
- net V_Out: now reaches C7.1, Q2.3, R3.1, U1.27 (VOUT), U1.28 (VOUT), U1.3 (VOUTA), U1.4 (CLN)
Changed lines of the file:
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@@
   (junction (at 160.02 63.5) (diameter 0) (color 0 0 0 0)
   )
-  (junction (at 160.02 105.41) (diameter 0) (color 0 0 0 0)
-  )
   (junction (at 73.66 60.96) (diameter 0) (color 0 0 0 0)
   )
@@
   (junction (at 73.66 69.85) (diameter 0) (color 0 0 0 0)
   )
+  (junction (at 163.83 63.5) (diameter 0) (color 0 0 0 0)
+  )
   (junction (at 135.89 73.66) (diameter 0) (color 0 0 0 0)
   )
+  (junction (at 160.02 104.14) (diameter 0) (color 0 0 0 0)
+  )
   (junction (at 74.93 97.79) (diameter 0) (color 0 0 0 0)
   )
@@
     (stroke (width 0) (type default) (color 0 0 0 0))
   )
-  (wire (pts (xy 160.02 101.6) (xy 160.02 105.41))
-    (stroke (width 0) (type default) (color 0 0 0 0))
-  )
   (wire (pts (xy 151.13 90.17) (xy 151.13 93.98))
     (stroke (width 0) (type default) (color 0 0 0 0))
@@
     (stroke (width 0) (type default) (color 0 0 0 0))
   )
+  (wire (pts (xy 160.02 104.14) (xy 166.37 104.14))
+    (stroke (width 0) (type default) (color 0 0 0 0))
+  )
   (wire (pts (xy 101.6 97.79) (xy 101.6 120.65))
     (stroke (width 0) (type default) (color 0 0 0 0))
@@
     (stroke (width 0) (type default) (color 0 0 0 0))
   )
-  (wire (pts (xy 102.87 60.96) (xy 142.24 60.96))
+  (wire (pts (xy 102.87 59.69) (xy 142.24 59.69))
     (stroke (width 0) (type default) (color 0 0 0 0))
   )
@@
     (stroke (width 0) (type default) (color 0 0 0 0))
   )
-  (wire (pts (xy 196.85 87.63) (xy 196.85 90.17))
-    (stroke (width 0) (type default) (color 0 0 0 0))
-  )
-  (wire (pts (xy 160.02 105.41) (xy 167.64 105.41))
-    (stroke (width 0) (type default) (color 0 0 0 0))
-  )
   (wire (pts (xy 134.62 100.33) (xy 140.97 100.33))
     (stroke (width 0) (type default) (color 0 0 0 0))
@@
     (stroke (width 0) (type default) (color 0 0 0 0))
   )
-  (wire (pts (xy 102.87 67.31) (xy 102.87 60.96))
+  (wire (pts (xy 102.87 59.69) (xy 102.87 67.31))
     (stroke (width 0) (type default) (color 0 0 0 0))
   )
@@
     (stroke (width 0) (type default) (color 0 0 0 0))
   )
+  (wire (pts (xy 160.02 104.14) (xy 160.02 106.68))
+    (stroke (width 0) (type default) (color 0 0 0 0))
+  )
   (wire (pts (xy 135.89 82.55) (xy 135.89 83.82))
     (stroke (width 0) (type default) (color 0 0 0 0))
@@
     (stroke (width 0) (type default) (color 0 0 0 0))
   )
-  (wire (pts (xy 142.24 60.96) (xy 142.24 67.31))
+  (wire (pts (xy 142.24 59.69) (xy 142.24 67.31))
     (stroke (width 0) (type default) (color 0 0 0 0))
   )
@@
     (stroke (width 0) (type default) (color 0 0 0 0))
   )
-  (wire (pts (xy 160.02 105.41) (xy 160.02 106.68))
-    (stroke (width 0) (type default) (color 0 0 0 0))
-  )
   (wire (pts (xy 104.14 69.85) (xy 97.79 69.85))
     (stroke (width 0) (type default) (color 0 0 0 0))
   )
+  (wire (pts (xy 160.02 101.6) (xy 160.02 104.14))
+    (stroke (width 0) (type default) (color 0 0 0 0))
+  )
   (wire (pts (xy 91.44 69.85) (xy 95.25 69.85))
     (stroke (width 0) (type default) (color 0 0 0 0))
   )
   (wire (pts (xy 72.39 60.96) (xy 73.66 60.96))
+    (stroke (width 0) (type default) (color 0 0 0 0))
+  )
+  (wire (pts (xy 163.83 63.5) (xy 170.18 63.5))
     (stroke (width 0) (type default) (color 0 0 0 0))
   )
@@
     (effects (font (size 1.27 1.27)) (justify right))
   )
-  (hierarchical_label "V_Bat" (shape input) (at 167.64 105.41 0)
+  (hierarchical_label "V_Bat" (shape input) (at 166.37 104.14 0)
+    (effects (font (size 1.27 1.27)) (justify left))
+  )
+  (hierarchical_label "V_Out" (shape input) (at 170.18 63.5 0)
     (effects (font (size 1.27 1.27)) (justify left))
   )
@@
       (effects (font (size 1.27 1.27)) (justify left))
     )
-    (property "Value" "C" (id 1) (at 88.9 84.455 0)
+    (property "Value" "1u" (id 1) (at 88.9 84.455 0)
       (effects (font (size 1.27 1.27)) (justify left))
     )
@@
     (in_bom yes) (on_board yes)
     (property "Reference" "R3" (id 0) (at 93.472 73.66 90))
-    (property "Value" "R" (id 1) (at 91.44 73.66 90))
+    (property "Value" "16m" (id 1) (at 88.9 73.66 90))
     (property "Footprint" "Resistor_SMD:R_0603_1608Metric_Pad0.98x0.95mm_HandSolder" (id 2) (at 89.662 73.66 90)
       (effects (font (size 1.27 1.27)) hide)
@@
       (effects (font (size 1.27 1.27)) (justify left))
     )
-    (property "Value" "C" (id 1) (at 164.465 69.85 0)
+    (property "Value" "10u" (id 1) (at 164.465 69.85 0)
       (effects (font (size 1.27 1.27)) (justify left))
     )
@@
     (in_bom yes) (on_board yes)
     (property "Reference" "L1" (id 0) (at 148.59 80.01 90))
-    (property "Value" "L" (id 1) (at 148.59 76.835 90))
+    (property "Value" "4.7u" (id 1) (at 148.59 76.835 90))
     (property "Footprint" "Inductor_SMD:L_0603_1608Metric_Pad1.05x0.95mm_HandSolder" (id 2) (at 148.59 78.74 0)
       (effects (font (size 1.27 1.27)) hide)
@@
       (effects (font (size 1.27 1.27)) (justify left))
     )
-    (property "Footprint" "2N7002:SOT23" (id 2) (at 160.02 85.09 0)
+    (property "Footprint" "Connectors_Cubesat_Custom:CubeSat_2n7002" (id 2) (at 160.02 85.09 0)
       (effects (font (size 1.27 1.27)) (justify left bottom) hide)
     )
@@
     (in_bom yes) (on_board yes)
     (property "Reference" "R4" (id 0) (at 91.948 99.06 90))
-    (property "Value" "R" (id 1) (at 93.98 99.06 90))
+    (property "Value" "63.4k" (id 1) (at 96.52 99.06 90))
     (property "Footprint" "Resistor_SMD:R_0603_1608Metric_Pad0.98x0.95mm_HandSolder" (id 2) (at 95.758 99.06 90)
       (effects (font (size 1.27 1.27)) hide)
@@
     (pin "2")
   )
-  (symbol (lib_id "power:GND") (at 196.85 87.63 180) (unit 1)
-    (in_bom yes) (on_board yes) (fields_autoplaced)
-    (property "Reference" "#PWR0110" (id 0) (at 196.85 81.28 0)
-      (effects (font (size 1.27 1.27)) hide)
-    )
-    (property "Value" "GND" (id 1) (at 196.85 82.55 0))
-    (property "Footprint" "" (id 2) (at 196.85 87.63 0)
-      (effects (font (size 1.27 1.27)) hide)
-    )
-    (property "Datasheet" "" (id 3) (at 196.85 87.63 0)
-      (effects (font (size 1.27 1.27)) hide)
-    )
-    (pin "1")
-  )
   (symbol (lib_id "Device:C") (at 160.02 110.49 0) (unit 1)
     (in_bom yes) (on_board yes)
@@
       (effects (font (size 1.27 1.27)) (justify left))
     )
-    (property "Value" "C" (id 1) (at 160.655 113.03 0)
+    (property "Value" "10u" (id 1) (at 160.655 113.03 0)
       (effects (font (size 1.27 1.27)) (justify left))
     )
@@
       (effects (font (size 1.27 1.27)) (justify left))
     )
-    (property "Value" "C" (id 1) (at 120.015 116.84 0)
+    (property "Value" "4.7u" (id 1) (at 120.015 116.84 0)
       (effects (font (size 1.27 1.27)) (justify left))
     )
@@
   (symbol (lib_id "power:GND") (at 137.16 114.3 0) (unit 1)
     (in_bom yes) (on_board yes) (fields_autoplaced)
-    (property "Reference" "#PWR0106" (id 0) (at 137.16 120.65 0)
+    (property "Reference" "#PWR08" (id 0) (at 137.16 120.65 0)
       (effects (font (size 1.27 1.27)) hide)
     )
@@
       (effects (font (size 1.27 1.27)) (justify left))
     )
-    (property "Value" "C_Polarized_US" (id 1) (at 58.42 61.595 0)
+    (property "Value" "150u" (id 1) (at 58.42 61.595 0)
       (effects (font (size 1.27 1.27)) (justify left))
     )
@@
     (pin "2")
   )
-  (symbol (lib_id "power:GNDPWR") (at 196.85 90.17 0) (unit 1)
-    (in_bom yes) (on_board yes) (fields_autoplaced)
-    (property "Reference" "#PWR0118" (id 0) (at 196.85 95.25 0)
-      (effects (font (size 1.27 1.27)) hide)
-    )
-    (property "Value" "GNDPWR" (id 1) (at 196.723 95.25 0))
-    (property "Footprint" "" (id 2) (at 196.85 91.44 0)
-      (effects (font (size 1.27 1.27)) hide)
-    )
-    (property "Datasheet" "" (id 3) (at 196.85 91.44 0)
-      (effects (font (size 1.27 1.27)) hide)
-    )
-    (pin "1")
-  )
   (symbol (lib_id "Device:R") (at 69.85 92.71 0) (unit 1)
     (in_bom yes) (on_board yes)
     (property "Reference" "R2" (id 0) (at 71.882 92.71 90))
-    (property "Value" "R" (id 1) (at 69.85 92.71 90))
+    (property "Value" "10k" (id 1) (at 67.31 92.71 90))
     (property "Footprint" "Resistor_SMD:R_0603_1608Metric_Pad0.98x0.95mm_HandSolder" (id 2) (at 68.072 92.71 90)
       (effects (font (size 1.27 1.27)) hide)
@@
       (effects (font (size 1.27 1.27)) (justify left))
     )
-    (property "Value" "C" (id 1) (at 142.875 73.66 0)
+    (property "Value" "22n" (id 1) (at 142.875 73.66 0)
       (effects (font (size 1.27 1.27)) (justify left))
     )
@@
       (effects (font (size 1.27 1.27)) (justify left))
     )
-    (property "Value" "C_Polarized_US" (id 1) (at 67.31 70.485 0)
+    (property "Value" "0.1u" (id 1) (at 67.31 70.485 0)
       (effects (font (size 1.27 1.27)) (justify left))
     )
@@
     (in_bom yes) (on_board yes)
     (property "Reference" "R1" (id 0) (at 68.58 62.992 90))
-    (property "Value" "R" (id 1) (at 68.58 60.96 90))
+    (property "Value" "2.5" (id 1) (at 68.58 60.96 90))
     (property "Footprint" "Resistor_SMD:R_0603_1608Metric_Pad0.98x0.95mm_HandSolder" (id 2) (at 68.58 59.182 90)
       (effects (font (size 1.27 1.27)) hide)
@@
     (in_bom yes) (on_board yes)
     (property "Reference" "R5" (id 0) (at 157.988 97.79 90))
-    (property "Value" "R" (id 1) (at 160.02 97.79 90))
+    (property "Value" "10m" (id 1) (at 162.56 97.79 90))
     (property "Footprint" "Resistor_SMD:R_0603_1608Metric_Pad0.98x0.95mm_HandSolder" (id 2) (at 161.798 97.79 90)
       (effects (font (size 1.27 1.27)) hide)
