File: Cubesat-Current/Power PCB/CubesatPwrBoard.kicad_sch (KiCad schematic)
At the start: 20 parts, among them J1 Conn_01x04_Female, J2 Conn_01x04_Female, J3 Conn_01x04_Female, J5 Conn_01x04_Female, J6 Conn_01x03_Female, J7 Conn_01x03_Female, J8 Conn_01x03_Female

Commit message: added to silkscreen and exported fabrication files
Parts:
- J5, J6, J7, J8: footprint Connector_PinSocket_2.54mm:PinSocket_1x04_P2.54mm_Vertical -> Connector_PinSocket_2.54mm:PinSocket_1x03_P2.54mm_Vertical
Changed lines of the file:
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@@
     (property "Reference" "J8" (id 0) (at 219.71 113.03 0))
     (property "Value" "Conn_01x03_Female" (id 1) (at 217.17 110.49 0))
-    (property "Footprint" "Connector_PinSocket_2.54mm:PinSocket_1x04_P2.54mm_Vertical" (id 2) (at 215.9 105.41 0)
+    (property "Footprint" "Connector_PinSocket_2.54mm:PinSocket_1x03_P2.54mm_Vertical" (id 2) (at 215.9 105.41 0)
       (effects (font (size 1.27 1.27)) hide)
     )
@@
     (property "Reference" "J7" (id 0) (at 219.71 82.55 0))
     (property "Value" "Conn_01x03_Female" (id 1) (at 217.17 80.01 0))
-    (property "Footprint" "Connector_PinSocket_2.54mm:PinSocket_1x04_P2.54mm_Vertical" (id 2) (at 215.9 74.93 0)
+    (property "Footprint" "Connector_PinSocket_2.54mm:PinSocket_1x03_P2.54mm_Vertical" (id 2) (at 215.9 74.93 0)
       (effects (font (size 1.27 1.27)) hide)
     )
@@
     (property "Reference" "J5" (id 0) (at 266.7 46.99 0))
     (property "Value" "Conn_01x04_Female" (id 1) (at 266.7 34.29 0))
-    (property "Footprint" "Connector_PinSocket_2.54mm:PinSocket_1x04_P2.54mm_Vertical" (id 2) (at 266.7 41.91 0)
+    (property "Footprint" "Connector_PinSocket_2.54mm:PinSocket_1x03_P2.54mm_Vertical" (id 2) (at 266.7 41.91 0)
       (effects (font (size 1.27 1.27)) hide)
     )
@@
     (property "Reference" "J6" (id 0) (at 218.44 52.07 0))
     (property "Value" "Conn_01x03_Female" (id 1) (at 215.9 49.53 0))
-    (property "Footprint" "Connector_PinSocket_2.54mm:PinSocket_1x04_P2.54mm_Vertical" (id 2) (at 214.63 44.45 0)
+    (property "Footprint" "Connector_PinSocket_2.54mm:PinSocket_1x03_P2.54mm_Vertical" (id 2) (at 214.63 44.45 0)
       (effects (font (size 1.27 1.27)) hide)
     )
@@
     )
     (path "/b96eb06c-d64f-41eb-9978-ba5d1bbedec4"
-      (reference "J5") (unit 1) (value "Conn_01x04_Female") (footprint "Connector_PinSocket_2.54mm:PinSocket_1x04_P2.54mm_Vertical")
+      (reference "J5") (unit 1) (value "Conn_01x04_Female") (footprint "Connector_PinSocket_2.54mm:PinSocket_1x03_P2.54mm_Vertical")
     )
     (path "/eb516b0b-cae1-4427-a0b9-096ca5da2e10"
-      (reference "J6") (unit 1) (value "Conn_01x03_Female") (footprint "Connector_PinSocket_2.54mm:PinSocket_1x04_P2.54mm_Vertical")
+      (reference "J6") (unit 1) (value "Conn_01x03_Female") (footprint "Connector_PinSocket_2.54mm:PinSocket_1x03_P2.54mm_Vertical")
     )
     (path "/6c45e2ce-632c-4e1d-ab74-73bdad14d9af"
-      (reference "J7") (unit 1) (value "Conn_01x03_Female") (footprint "Connector_PinSocket_2.54mm:PinSocket_1x04_P2.54mm_Vertical")
+      (reference "J7") (unit 1) (value "Conn_01x03_Female") (footprint "Connector_PinSocket_2.54mm:PinSocket_1x03_P2.54mm_Vertical")
     )
     (path "/5156cae7-9267-423b-905d-ea8c4e454f3c"
-      (reference "J8") (unit 1) (value "Conn_01x03_Female") (footprint "Connector_PinSocket_2.54mm:PinSocket_1x04_P2.54mm_Vertical")
+      (reference "J8") (unit 1) (value "Conn_01x03_Female") (footprint "Connector_PinSocket_2.54mm:PinSocket_1x03_P2.54mm_Vertical")
     )
     (path "/cf1aff82-9d0a-48d8-ab59-8548d6686ba1/e6dc0141-26d6-4149-b18d-3c71f4483f5c"

Commit message: Updating to revision 5.0
Parts:
- removed BT1, BT2, BT3, BT4: 254TR, 254TR:BAT_254TR, symbol 254TR:254TR
- removed J3: Conn_01x04_Female, Connector_PinSocket_2.54mm:PinSocket_1x04_P2.54mm_Vertical, symbol Connector:Conn_01x04_Female
- removed J5: Conn_01x04_Female, Connector_PinSocket_2.54mm:PinSocket_1x03_P2.54mm_Vertical, symbol Connector:Conn_01x03_Female
- removed J6, J8: Conn_01x03_Female, Connector_PinSocket_2.54mm:PinSocket_1x03_P2.54mm_Vertical, symbol Connector:Conn_01x03_Female
- removed TH2: Thermistor_NTC, Resistor_SMD:R_0402_1005Metric_Pad0.72x0.64mm_HandSolder, symbol Device:Thermistor_NTC
- added J3, J4: 254TR, 254TR:BAT_254TR, symbol 254TR:254TR
- added J7: Conn_01x03_Female, Connectors_Cubesat_Custom:CubeSat_Conn_3x01_P2.54mm, symbol Connector:Conn_01x03_Female
- added J9: Conn_01x02_Female, Connectors_Cubesat_Custom:CubeSat_Conn_2x01_P2.54mm, symbol Connector:Conn_01x02_Female
- H1: renamed from H2; footprint MountingHole:MountingHole_4.3mm_M4_DIN965_Pad -> Connectors_Cubesat_Custom:CubeSat_MountingHole_M4
- H2: renamed from H4; footprint MountingHole:MountingHole_4.3mm_M4_DIN965_Pad -> Connectors_Cubesat_Custom:CubeSat_MountingHole_M4
- H3: renamed from H1; footprint MountingHole:MountingHole_4.3mm_M4_DIN965_Pad -> Connectors_Cubesat_Custom:CubeSat_MountingHole_M4
- H4: renamed from H3; footprint MountingHole:MountingHole_4.3mm_M4_DIN965_Pad -> Connectors_Cubesat_Custom:CubeSat_MountingHole_M4
- J1, J2: footprint Connector_PinSocket_2.54mm:PinSocket_1x04_P2.54mm_Vertical -> Connectors_Cubesat_Custom:CubeSat_Conn_4x01_P2.54mm
- J8: renamed from J7; footprint Connector_PinSocket_2.54mm:PinSocket_1x03_P2.54mm_Vertical -> Connectors_Cubesat_Custom:CubeSat_Conn_3x01_P2.54mm
- renumbered BT5 to J5, BT6 to J6, TH3 to TH2
Connections:
- net GND: now also J4.P1_1, J4.P1_2
- net V_Reg_3.3_5V3/Vout: now also J9.2 (Pin_2)
- net Bat_Reg_1/DVCC renamed Bat_Reg_4/DVCC
- net Bat_Reg_1/SCL renamed Bat_Reg_4/SCL
- net Bat_Reg_1/SDA renamed Bat_Reg_4/SDA
- net Bat_Reg_1/TH renamed Bat_Reg_4/TH
- net Bat_Reg_1//SMBALERT renamed Bat_Reg_4//SMBALERT
- new net Bat_Reg_4/V_Bat: J3.P1_1, J3.P1_2
- new net V_Reg_3.3_5V4/#SHDN: J7.3 (Pin_3)
- new net V_Reg_3.3_5V4/#STBY: J7.2 (Pin_2)
- new net V_Reg_3.3_5V4/3/#5: J7.1 (Pin_1)
- new net V_Reg_3.3_5V4/Vout: J9.1 (Pin_1)
Other:
- removed sheet Bat_Reg_1
- removed sheet Bat_Reg_2
- removed sheet V_Reg_3.3_5V1
- removed sheet V_Reg_3.3_5V2
- added sheet Bat_Reg_4 (Bat_Reg_1.kicad_sch)
- added sheet V_Reg_3.3_5V4 (V_Reg_3.3V.kicad_sch)
- sheet Bat_Reg_3 ports: added V_Out; removed none
- sheet Solar_Panels ports: added none; removed V_R3
- note removed: "Each battery gets its own PMIC regulating voltage and its own I2C port for management"
- note removed: "Will add ICs to regulate battery output so that voltage output is always 3.3V/5V"
- moved on the sheet: H2, J2, J5, J6, J8, TH2
