File: Cubesat-Current/Power PCB/Solar_Panels.kicad_sch (KiCad schematic)
At the start: 9 parts, among them J10 S1, J11 S2, J12 S3, J13 S4, J14 S5, J15 S6

Commit message: Updating to revision 5.0
Parts:
- removed D2: D_Schottky_Small, CUS520,H3F:DIO_CUS520,H3F, symbol Device:D_Schottky_Small
- D1: footprint CUS520,H3F:DIO_CUS520,H3F -> Connectors_Cubesat_Custom:CubeSat_DIO_CUS520,H3f
- D2: renamed from D3; footprint CUS520,H3F:DIO_CUS520,H3F -> Connectors_Cubesat_Custom:CubeSat_DIO_CUS520,H3f
- J10, J11, J12, J13, J14, J15: footprint Connector_PinSocket_2.54mm:PinSocket_2x03_P2.54mm_Vertical -> Connectors_Cubesat_Custom:CubeSat_Conn_2x02_P2.54mm; symbol Connector:Conn_01x06_Female -> Connector:Conn_01x04_Female
Connections:
- net GND: now also J10.2 (Pin_2), J10.4 (Pin_4), J11.2 (Pin_2), J11.4 (Pin_4), J12.2 (Pin_2), J12.4 (Pin_4), J13.2 (Pin_2), J13.4 (Pin_4), J14.2 (Pin_2), J14.4 (Pin_4), J15.2 (Pin_2), J15.4 (Pin_4); no longer J10.1 (Pin_1), J10.3 (Pin_3), J10.5 (Pin_5), J11.1 (Pin_1), J11.3 (Pin_3), J11.5 (Pin_5), J12.1 (Pin_1), J12.3 (Pin_3), J12.5 (Pin_5), J13.1 (Pin_1), J13.3 (Pin_3), J13.5 (Pin_5), J14.1 (Pin_1), J14.3 (Pin_3), J14.5 (Pin_5), J15.1 (Pin_1), J15.3 (Pin_3), J15.5 (Pin_5)
- new net: D2.2 (A), J10.1 (Pin_1), J11.1 (Pin_1), J12.1 (Pin_1), J13.1 (Pin_1), J14.1 (Pin_1), J15.1 (Pin_1)
- new net: D1.2 (A), J10.3 (Pin_3), J11.3 (Pin_3), J12.3 (Pin_3), J13.3 (Pin_3), J14.3 (Pin_3), J15.3 (Pin_3)
