File: Cubesat-Current/Power PCB/V_Reg_3.3V.kicad_sch (KiCad schematic)
At the start: 5 parts, among them U5 MAX710ESE+T

Commit message: Updating to revision 5.0
Parts:
- C15: renamed from C29; value C_Polarized_US -> 4.7u
- C16: renamed from C30; value C_Polarized_US -> 100u; footprint Capacitor_SMD:C_0603_1608Metric_Pad1.08x0.95mm_HandSolder -> Capacitor_SMD:C_0805_2012Metric_Pad1.18x1.45mm_HandSolder
- D3: renamed from D5; footprint Diode_SMD:D_0603_1608Metric_Pad1.05x0.95mm_HandSolder -> Connectors_Cubesat_Custom:CubeSat_Diode_SOT_882
- L3: renamed from L5; value L -> 22u
- renumbered U5 to U3
Changed lines of the file:
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@@
   (symbol (lib_id "power:GND") (at 69.85 62.23 0) (unit 1)
     (in_bom yes) (on_board yes) (fields_autoplaced)
-    (property "Reference" "#PWR01" (id 0) (at 69.85 68.58 0)
+    (property "Reference" "#PWR010" (id 0) (at 69.85 68.58 0)
       (effects (font (size 1.27 1.27)) hide)
     )
@@
   (symbol (lib_id "Device:C_Polarized_US") (at 152.4 62.23 0) (unit 1)
     (in_bom yes) (on_board yes)
-    (property "Reference" "C30" (id 0) (at 153.035 59.69 0)
+    (property "Reference" "C16" (id 0) (at 153.035 59.69 0)
       (effects (font (size 1.27 1.27)) (justify left))
     )
-    (property "Value" "C_Polarized_US" (id 1) (at 153.035 64.77 0)
+    (property "Value" "100u" (id 1) (at 153.035 64.77 0)
       (effects (font (size 1.27 1.27)) (justify left))
     )
-    (property "Footprint" "Capacitor_SMD:C_0603_1608Metric_Pad1.08x0.95mm_HandSolder" (id 2) (at 152.4 62.23 0)
+    (property "Footprint" "Capacitor_SMD:C_0805_2012Metric_Pad1.18x1.45mm_HandSolder" (id 2) (at 152.4 62.23 0)
       (effects (font (size 1.27 1.27)) hide)
     )
@@
   (symbol (lib_id "power:PWR_FLAG") (at 170.18 43.18 180) (unit 1)
     (in_bom yes) (on_board yes) (fields_autoplaced)
-    (property "Reference" "#FLG0101" (id 0) (at 170.18 45.085 0)
+    (property "Reference" "#FLG01" (id 0) (at 170.18 45.085 0)
       (effects (font (size 1.27 1.27)) hide)
     )
@@
   (symbol (lib_id "Device:C_Polarized_US") (at 135.89 73.66 0) (unit 1)
     (in_bom yes) (on_board yes)
-    (property "Reference" "C29" (id 0) (at 136.525 71.12 0)
+    (property "Reference" "C15" (id 0) (at 136.525 71.12 0)
       (effects (font (size 1.27 1.27)) (justify left))
     )
-    (property "Value" "C_Polarized_US" (id 1) (at 136.525 76.2 0)
+    (property "Value" "4.7u" (id 1) (at 136.525 76.2 0)
       (effects (font (size 1.27 1.27)) (justify left))
     )
@@
   (symbol (lib_id "Device:D_Schottky") (at 121.92 54.61 180) (unit 1)
     (in_bom yes) (on_board yes) (fields_autoplaced)
-    (property "Reference" "D5" (id 0) (at 122.2375 48.26 0))
+    (property "Reference" "D3" (id 0) (at 122.2375 48.26 0))
     (property "Value" "D_Schottky" (id 1) (at 122.2375 50.8 0))
-    (property "Footprint" "Diode_SMD:D_0603_1608Metric_Pad1.05x0.95mm_HandSolder" (id 2) (at 121.92 54.61 0)
+    (property "Footprint" "Connectors_Cubesat_Custom:CubeSat_Diode_SOT_882" (id 2) (at 121.92 54.61 0)
       (effects (font (size 1.27 1.27)) hide)
     )
@@
   (symbol (lib_id "power:GND") (at 152.4 66.04 0) (unit 1)
     (in_bom yes) (on_board yes) (fields_autoplaced)
-    (property "Reference" "#PWR05" (id 0) (at 152.4 72.39 0)
+    (property "Reference" "#PWR012" (id 0) (at 152.4 72.39 0)
       (effects (font (size 1.27 1.27)) hide)
     )
@@
   (symbol (lib_id "Device:L") (at 99.06 43.18 90) (unit 1)
     (in_bom yes) (on_board yes)
-    (property "Reference" "L5" (id 0) (at 99.06 44.45 90))
-    (property "Value" "L" (id 1) (at 99.06 41.275 90))
+    (property "Reference" "L3" (id 0) (at 99.06 44.45 90))
+    (property "Value" "22u" (id 1) (at 99.06 41.275 90))
     (property "Footprint" "Inductor_SMD:L_0603_1608Metric_Pad1.05x0.95mm_HandSolder" (id 2) (at 99.06 43.18 0)
       (effects (font (size 1.27 1.27)) hide)
@@
   (symbol (lib_id "MAX710ESE_T:MAX710ESE+T") (at 96.52 73.66 0) (unit 1)
     (in_bom yes) (on_board yes) (fields_autoplaced)
-    (property "Reference" "U5" (id 0) (at 96.52 45.72 0))
+    (property "Reference" "U3" (id 0) (at 96.52 45.72 0))
     (property "Value" "MAX710ESE+T" (id 1) (at 96.52 48.26 0))
     (property "Footprint" "MAX710ESE:SOIC127P600X175-16N" (id 2) (at 86.36 99.06 0)
@@
   (symbol (lib_id "power:GND") (at 170.18 40.64 180) (unit 1)
     (in_bom yes) (on_board yes) (fields_autoplaced)
-    (property "Reference" "#PWR04" (id 0) (at 170.18 34.29 0)
+    (property "Reference" "#PWR013" (id 0) (at 170.18 34.29 0)
       (effects (font (size 1.27 1.27)) hide)
     )
@@
   (symbol (lib_id "power:GND") (at 135.89 77.47 0) (unit 1)
     (in_bom yes) (on_board yes) (fields_autoplaced)
-    (property "Reference" "#PWR03" (id 0) (at 135.89 83.82 0)
+    (property "Reference" "#PWR011" (id 0) (at 135.89 83.82 0)
       (effects (font (size 1.27 1.27)) hide)
     )
