File: Power PCB/CubesatPwrBoard.kicad_pcb (KiCad board)
At the start: 2 copper layers, 90 x 96 mm, 65 parts, among them J1 Conn_01x04_Female, J10 S1, J11 S2, J12 S3, J13 S4, J14 S5, J15 S6, J2 Conn_01x04_Female, J3 254TR, J4 254TR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

Commit message: Added gerbers
Other:
- board text added: "0.1u"
- board text added: "100u"
- board text added: "10k"
- board text added: "10m"
- board text added: "10u"
- board text added: "150u"
- board text added: "16m"
- board text added: "1u"
- board text added: "2.5"
- board text added: "22n"
- board text added: "22u"
- board text added: "2N7"
- board text added: "4.7u"
- board text added: "63.4k"
- board text added: "BAS"
- board text added: "CUS"
- board text added: "TQM"
